Commit message: novo modelo atualizado do robô

File: src/trekking/description/robot_core.urdf.xacro (robot description, xacro)
@@ -29,5 +29,5 @@
             <origin xyz="0 0 0.07" rpy="0 0 0"/>
             <geometry>
-                <box size="0.4 0.2 0.1"/>
+                <box size="0.37 0.2 0.1"/>
             </geometry>
             <material name="black"/>
@@ -36,5 +36,5 @@
             <origin xyz="0 0 0.07" rpy="0 0 0"/>
             <geometry>
-                <box size="0.4 0.2 0.1"/>
+                <box size="0.37 0.2 0.1"/>
             </geometry>
         </collision>
@@ -68,5 +68,5 @@
         <parent link="chassis"/>
         <child link="laser_frame"/>
-        <origin xyz="0.1 0 0.131" rpy="0 0 0"/>
+        <origin xyz="0 0 0" rpy="0 0 -1.57"/>
     </joint>
     <link name="left_front_wheel_link">
@@ -93,5 +93,5 @@
         <parent link="base_link"/>
         <child link="left_front_wheel_link"/>
-        <origin xyz="0.165 0.13 0.03" rpy="-1.57 0 0"/>
+        <origin xyz="0.105 0.135 0.03" rpy="-1.57 0 0"/>
         <axis xyz="0 0 -1"/>
     </joint>
@@ -119,5 +119,5 @@
         <parent link="base_link"/>
         <child link="right_front_wheel_link"/>
-        <origin xyz="0.165 -0.13 0.03" rpy="1.57 0 0"/>
+        <origin xyz="0.105 -0.135 0.03" rpy="1.57 0 0"/>
         <axis xyz="0 0 -1"/>
     </joint>
@@ -145,5 +145,5 @@
         <parent link="base_link"/>
         <child link="left_rear_wheel_link"/>
-        <origin xyz="-0.165 0.13 0.03" rpy="-1.57 0 0"/>
+        <origin xyz="-0.105 0.135 0.03" rpy="-1.57 0 0"/>
         <axis xyz="0 0 -1"/>
     </joint>
@@ -171,5 +171,5 @@
         <parent link="base_link"/>
         <child link="right_rear_wheel_link"/>
-        <origin xyz="-0.165 -0.13 0.03" rpy="1.57 0 0"/>
+        <origin xyz="-0.105 -0.135 0.03" rpy="1.57 0 0"/>
         <axis xyz="0 0 -1"/>
     </joint>

Commit message: novo modelo atualizado do robô

File: src/trekking/description/robot_core.urdf.xacro (robot description, xacro)
@@ -68,5 +68,5 @@
         <parent link="chassis"/>
         <child link="laser_frame"/>
-        <origin xyz="0 0 0" rpy="0 0 -1.57"/>
+        <origin xyz="0.1 0 0.13" rpy="0 0 0"/>
     </joint>
     <link name="left_front_wheel_link">

Commit message: Melhor vizualizador RViz

File: src/trekking/description/robot_core.urdf.xacro (robot description, xacro)
@@ -68,5 +68,5 @@
         <parent link="chassis"/>
         <child link="laser_frame"/>
-        <origin xyz="0.1 0 0.13" rpy="0 0 0"/>
+        <origin xyz="0 0 0.13" rpy="0 0 0"/>
     </joint>
     <link name="left_front_wheel_link">
